File: pcb/mic_array/array.kicad_sch (KiCad schematic)
At the start: 26 parts, among them J1 M55-7002042R, J2 M55-7002042R

Commit message: JLCPCB ready
Parts:
- J1, J2: LCSC C17365015 -> C7503099
Other:
- note added: "Author: Andrés CALDERÓN"
- note added: "Top page, microphone array"
- note added: "email: andresfcalderon@gmail.com"
- note added: "https://github.com/Iari-Lab/OpenAcousticCamera"
Changed lines of the file:
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@@
 		)
 	)
+	(text "email: andresfcalderon@gmail.com\n"
+		(exclude_from_sim no)
+		(at 319.278 260.35 0)
+		(effects
+			(font
+				(size 1.27 1.27)
+				(thickness 0.254)
+				(bold yes)
+			)
+		)
+	)
+	(text "Author: Andrés CALDERÓN"
+		(exclude_from_sim no)
+		(at 314.96 256.794 0)
+		(effects
+			(font
+				(size 1.27 1.27)
+				(thickness 0.254)
+				(bold yes)
+			)
+		)
+	)
+	(text "https://github.com/Iari-Lab/OpenAcousticCamera\n"
+		(exclude_from_sim no)
+		(at 326.898 263.906 0)
+		(effects
+			(font
+				(size 1.27 1.27)
+				(thickness 0.254)
+				(bold yes)
+			)
+		)
+	)
+	(text "Top page, microphone array"
+		(exclude_from_sim no)
+		(at 324.612 276.606 0)
+		(effects
+			(font
+				(size 1.27 1.27)
+				(thickness 0.254)
+				(bold yes)
+			)
+		)
+	)
 	(junction
 		(at 53.34 228.6)
@@
 			)
 		)
-		(property "LCSC" "C17365015"
+		(property "LCSC" "C7503099"
 			(at 124.46 228.6 90)
 			(effects
@@
 			)
 		)
-		(property "LCSC" "C17365015"
+		(property "LCSC" "C7503099"
 			(at 50.8 228.6 90)
 			(effects
