File: pcb/mic_array/mics.kicad_sch (KiCad schematic)
At the start: 180 parts, among them M0 SPH0641LU4H-1, M1 SPH0641LU4H-1, M10 SPH0641LU4H-1, M11 SPH0641LU4H-1, M12 SPH0641LU4H-1, M13 SPH0641LU4H-1, M14 SPH0641LU4H-1, M15 SPH0641LU4H-1, M16 SPH0641LU4H-1, M17 SPH0641LU4H-1, M18 SPH0641LU4H-1, M19 SPH0641LU4H-1, M2 SPH0641LU4H-1, M20 SPH0641LU4H-1, M21 SPH0641LU4H-1, M22 SPH0641LU4H-1, M23 SPH0641LU4H-1, M24 SPH0641LU4H-1, M25 SPH0641LU4H-1, M26 SPH0641LU4H-1, M27 SPH0641LU4H-1, M28 SPH0641LU4H-1, M29 SPH0641LU4H-1, M3 SPH0641LU4H-1, M30 SPH0641LU4H-1, M31 SPH0641LU4H-1, M32 SPH0641LU4H-1, M33 SPH0641LU4H-1, M34 SPH0641LU4H-1, M35 SPH0641LU4H-1, M36 SPH0641LU4H-1, M37 SPH0641LU4H-1, M38 SPH0641LU4H-1, M39 SPH0641LU4H-1, M4 SPH0641LU4H-1, M40 SPH0641LU4H-1, M41 SPH0641LU4H-1, M42 SPH0641LU4H-1, M43 SPH0641LU4H-1, M44 SPH0641LU4H-1, M45 SPH0641LU4H-1, M46 SPH0641LU4H-1, M47 SPH0641LU4H-1, M48 SPH0641LU4H-1, M49 SPH0641LU4H-1, M5 SPH0641LU4H-1, M50 SPH0641LU4H-1, M51 SPH0641LU4H-1, M52 SPH0641LU4H-1, M53 SPH0641LU4H-1, M54 SPH0641LU4H-1, M55 SPH0641LU4H-1, M56 SPH0641LU4H-1, M57 SPH0641LU4H-1, M58 SPH0641LU4H-1, M59 SPH0641LU4H-1, M6 SPH0641LU4H-1, M7 SPH0641LU4H-1, M8 SPH0641LU4H-1, M9 SPH0641LU4H-1

Commit message: JLCPCB ready
Other:
- note added: "Author: Andrés CALDERÓN"
- note added: "Microphones"
- note added: "email: andresfcalderon@gmail.com"
- note added: "https://github.com/Iari-Lab/OpenAcousticCamera"
Changed lines of the file:
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@@
 	(generator_version "9.0")
 	(paper "A2")
+	(text "email: andresfcalderon@gmail.com\n"
+		(exclude_from_sim no)
+		(at 493.268 384.048 0)
+		(effects
+			(font
+				(size 1.27 1.27)
+				(thickness 0.254)
+				(bold yes)
+			)
+		)
+	)
+	(text "Author: Andrés CALDERÓN"
+		(exclude_from_sim no)
+		(at 488.95 380.492 0)
+		(effects
+			(font
+				(size 1.27 1.27)
+				(thickness 0.254)
+				(bold yes)
+			)
+		)
+	)
+	(text "https://github.com/Iari-Lab/OpenAcousticCamera\n"
+		(exclude_from_sim no)
+		(at 500.888 387.604 0)
+		(effects
+			(font
+				(size 1.27 1.27)
+				(thickness 0.254)
+				(bold yes)
+			)
+		)
+	)
+	(text "Microphones"
+		(exclude_from_sim no)
+		(at 498.348 399.542 0)
+		(effects
+			(font
+				(size 1.27 1.27)
+				(thickness 0.254)
+				(bold yes)
+			)
+		)
+	)
 	(junction
 		(at 318.77 240.03)
