File: pcb/controller_zynq/PSU.kicad_sch (KiCad schematic)
At the start: 32 parts, among them J2 USB_C_Receptacle_USB2.0, M3 AG9905-MTB, Q1 DMG2305UX, Q2 BCM857BS, U8 TVS1401DRBR

Commit message: fixing diodes
Connections:
- net POE_PR12: now also D3.3; no longer D3.4 (-)
- net POE_PR36: now also D3.1; no longer D3.2 (+)
- net POE_PR45: now also D4.3; no longer D4.4 (-)
- net POE_PR78: now also D4.1; no longer D4.2 (+)
- net at D1.2 (A2), L6.1, R8.1: now also D3.4 (-), D4.4 (-); no longer D3.1, D4.1
- net at D1.1 (A1), L3.1, R7.1: now also D3.2 (+), D4.2 (+); no longer D3.3, D4.3
Other:
- moved on the sheet: D3, D4
Changed lines of the file:
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@@
 	(symbol
 		(lib_id "SBR05M100BLP:SBR05M100BLP-7")
-		(at 26.67 99.06 0)
+		(at 26.67 99.06 90)
 		(unit 1)
 		(exclude_from_sim no)
@@
 		(dnp no)
 		(property "Reference" "D3"
-			(at 41.91 92.7414 0)
+			(at 20.3514 83.82 0)
 			(effects
 				(font
@@
 		)
 		(property "Value" "SBR05M100BLP-7"
-			(at 33.782 105.156 0)
+			(at 32.766 91.948 0)
 			(effects
 				(font
@@
 		)
 		(property "Footprint" "smd:RECTIFIER_SBR05M100BLP-7"
-			(at 27.686 83.058 0)
+			(at 10.668 98.044 0)
 			(effects
 				(font
@@
 	(symbol
 		(lib_id "SBR05M100BLP:SBR05M100BLP-7")
-		(at 54.61 99.06 0)
+		(at 54.61 99.06 90)
 		(unit 1)
 		(exclude_from_sim no)
@@
 		(dnp no)
 		(property "Reference" "D4"
-			(at 69.85 92.7414 0)
+			(at 48.2914 83.82 0)
 			(effects
 				(font
@@
 		)
 		(property "Value" "SBR05M100BLP-7"
-			(at 61.722 105.156 0)
+			(at 60.706 91.948 0)
 			(effects
 				(font
@@
 		)
 		(property "Footprint" "smd:RECTIFIER_SBR05M100BLP-7"
-			(at 55.626 83.058 0)
-			(effects
-				(font
+			(at 38.608 98.044 0)
+			(effects
+				(font
