File: pcb/controller_zynq/controller.kicad_pcb (KiCad board)
At the start: 6 copper layers, 94 x 78 mm, 130 parts, among them J1 USB1125-GF-B_REVA, J2 USB_C_Receptacle_USB2.0, J3 473092651, J4 ARJ-146, J5 TRS_LINE_OUT, J6 CON-SMA-EDGE-S, J7 95278-101A12LF, J8 CON-SMA-EDGE-S, J9 Conn_02x02_Odd_Even, M1 MYC-C7Z0XX_M1, M2 MYC-C7Z0XX_M1, M3 AG9905-MTB, Q1 DMG2305UX, Q2 BCM857BS, SW1 FPGA reset, U1 NVT4858HKZ, U10 PCM5101A, U11 TXS0102DQMR, U12 TXS0102DQMR, U2 74AHC1G04, U3 HSP051-4N10, U4 HSP051-4N10, U5 TXS0102DQMR, U6 SN74LVC2G07DBVR, U7 LDL212PV33R, U8 TVS1401DRBR, U9 TXS0102DQMR

Commit message: fixing diodes
Parts:
- moved L3 0.66 mm to (95.9, 123.4)
- moved L4 0.66 mm to (95.9, 125.1)
- moved L5 0.66 mm to (95.9, 126.9)
- moved R7 0.49 mm to (93.3, 124.1)
- moved D4 0.44 mm to (99.9, 124.5), turned to 0 degrees
- moved L6 0.26 mm to (107.6, 123.0)
- moved L7 0.26 mm to (107.6, 124.7)
- moved L8 0.26 mm to (107.6, 126.5)
- moved D3 0.25 mm to (103.8, 124.5), turned to 0 degrees
- moved C29 0.22 mm to (93.0, 128.5)
Connections:
- D3 pad 1: Net-(D1-A2) -> /Ethernet/POE_PR36
- D3 pad 2: /Ethernet/POE_PR36 -> Net-(D1-A1)
- D3 pad 3: Net-(D1-A1) -> /Ethernet/POE_PR12
- D3 pad 4: /Ethernet/POE_PR12 -> Net-(D1-A2)
- D4 pad 1: Net-(D1-A2) -> /Ethernet/POE_PR78
- D4 pad 2: /Ethernet/POE_PR78 -> Net-(D1-A1)
- D4 pad 3: Net-(D1-A1) -> /Ethernet/POE_PR45
- D4 pad 4: /Ethernet/POE_PR45 -> Net-(D1-A2)
Routing:
- net /PSU/PoE_VIN+: track 5.16 -> 1.09 mm
- net /Ethernet/POE_PR12: track 30.2 -> 26.9 mm, vias 1 -> 2
- net Net-(D1-A2): track 26.1 -> 29.2 mm, vias 0 -> 2
- net /SOM/D22: track 29.4 -> 28.7 mm
